File: AudioAmp.kicad_sch (KiCad schematic)
At the start: 59 parts, among them J1 ACJS-MHOM, J2 ACJS-MHOM, Q1 MJE182G, Q12 MMBT5401, Q13 MMBT5401, Q2 MJE172G, Q3 MMBT5551(RANGE:200-300), Q9 MMBT5551(RANGE:200-300)

Commit message: CHA: Syncronität SHA / PCB
Parts:
- renumbered H5 to GND1, H7 to GND2, J1 to Jack-IN1, J2 to Jack-OUT1, MNT1 to MNT/GND1, MNT2 to MNT/GND2, MNT3 to MNT/GND3, MNT4 to MNT/GND4, H9 to Rear-IN1, H1 to Rear-OUT1, H2 to Tip-IN1, H8 to Tip-OUT1, H3 to VCC+1, H4 to VCC-1
Changed lines of the file:
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@@
 		(dnp yes)
 		(fields_autoplaced yes)
-		(property "Reference" "MNT4"
+		(property "Reference" "MNT/GND4"
 			(at 87.63 147.32 90)
 			(effects
@@
 			(project "AudioAmp"
 				(path "/c5a26e6d-aabf-49ab-a44e-c2ec87fd373d"
-					(reference "MNT4")
+					(reference "MNT/GND4")
 					(unit 1)
 				)
@@
 		(dnp yes)
 		(fields_autoplaced yes)
-		(property "Reference" "H8"
+		(property "Reference" "Tip-OUT1"
 			(at 265.43 73.6599 0)
 			(effects
@@
 			(project ""
 				(path "/c5a26e6d-aabf-49ab-a44e-c2ec87fd373d"
-					(reference "H8")
+					(reference "Tip-OUT1")
 					(unit 1)
 				)
@@
 		(dnp yes)
 		(fields_autoplaced yes)
-		(property "Reference" "H4"
+		(property "Reference" "VCC-1"
 			(at 265.43 126.9999 90)
 			(effects
@@
 			(project ""
 				(path "/c5a26e6d-aabf-49ab-a44e-c2ec87fd373d"
-					(reference "H4")
+					(reference "VCC-1")
 					(unit 1)
 				)
@@
 		(dnp yes)
 		(fields_autoplaced yes)
-		(property "Reference" "H5"
+		(property "Reference" "GND1"
 			(at 44.45 99.06 90)
 			(effects
@@
 			(project ""
 				(path "/c5a26e6d-aabf-49ab-a44e-c2ec87fd373d"
-					(reference "H5")
+					(reference "GND1")
 					(unit 1)
 				)
@@
 		(dnp yes)
 		(fields_autoplaced yes)
-		(property "Reference" "H1"
+		(property "Reference" "Rear-OUT1"
 			(at 267.97 77.47 90)
 			(effects
@@
 			(project ""
 				(path "/c5a26e6d-aabf-49ab-a44e-c2ec87fd373d"
-					(reference "H1")
+					(reference "Rear-OUT1")
 					(unit 1)
 				)
@@
 		(dnp yes)
 		(fields_autoplaced yes)
-		(property "Reference" "MNT3"
+		(property "Reference" "MNT/GND3"
 			(at 62.23 140.97 90)
 			(effects
@@
 			(project "AudioAmp"
 				(path "/c5a26e6d-aabf-49ab-a44e-c2ec87fd373d"
-					(reference "MNT3")
+					(reference "MNT/GND3")
 					(unit 1)
 				)
@@
 		(dnp yes)
 		(fields_autoplaced yes)
-		(property "Reference" "H3"
+		(property "Reference" "VCC+1"
 			(at 265.43 49.5299 90)
 			(effects
@@
 			(project ""
 				(path "/c5a26e6d-aabf-49ab-a44e-c2ec87fd373d"
-					(reference "H3")
+					(reference "VCC+1")
 					(unit 1)
 				)
@@
 		(dnp yes)
 		(fields_autoplaced yes)
-		(property "Reference" "H2"
+		(property "Reference" "Tip-IN1"
 			(at 43.18 76.2 90)
 			(effects
@@
 			(project ""
 				(path "/c5a26e6d-aabf-49ab-a44e-c2ec87fd373d"
-					(reference "H2")
+					(reference "Tip-IN1")
 					(unit 1)
 				)
@@
 		(dnp yes)
 		(fields_autoplaced yes)
-		(property "Reference" "MNT1"
+		(property "Reference" "MNT/GND1"
 			(at 45.72 119.38 90)
 			(effects
@@
 			(project "AudioAmp"
 				(path "/c5a26e6d-aabf-49ab-a44e-c2ec87fd373d"
-					(reference "MNT1")
+					(reference "MNT/GND1")
 					(unit 1)
 				)
@@
 		(dnp yes)
 		(fields_autoplaced yes)
-		(property "Reference" "H9"
+		(property "Reference" "Rear-IN1"
 			(at 38.1 92.7099 90)
 			(effects
@@
 			(project ""
 				(path "/c5a26e6d-aabf-49ab-a44e-c2ec87fd373d"
-					(reference "H9")
+					(reference "Rear-IN1")
 					(unit 1)
 				)
@@
 		(dnp yes)
 		(fields_autoplaced yes)
-		(property "Reference" "MNT2"
+		(property "Reference" "MNT/GND2"
 			(at 58.42 127 90)
 			(effects
@@
 			(project "AudioAmp"
 				(path "/c5a26e6d-aabf-49ab-a44e-c2ec87fd373d"
-					(reference "MNT2")
+					(reference "MNT/GND2")
 					(unit 1)
 				)
@@
 		(dnp yes)
 		(fields_autoplaced yes)
-		(property "Reference" "H7"
+		(property "Reference" "GND2"
 			(at 269.24 100.3299 90)
 			(effects
@@
 			(project ""
 				(path "/c5a26e6d-aabf-49ab-a44e-c2ec87fd373d"
-					(reference "H7")
+					(reference "GND2")
 					(unit 1)
 				)
@@
 		(dnp no)
 		(fields_autoplaced yes)
-		(property "Reference" "J2"
+		(property "Reference" "Jack-OUT1"
 			(at 284.48 81.2799 0)
 			(effects
@@
 			(project ""
 				(path "/c5a26e6d-aabf-49ab-a44e-c2ec87fd373d"
-					(reference "J2")
+					(reference "Jack-OUT1")
 					(unit 1)
 				)
@@
 		(on_board yes)
 		(dnp no)
-		(property "Reference" "J1"
+		(property "Reference" "Jack-IN1"
 			(at 18.415 105.41 0)
 			(effects
@@
 			(project ""
 				(path "/c5a26e6d-aabf-49ab-a44e-c2ec87fd373d"
-					(reference "J1")
+					(reference "Jack-IN1")
 					(unit 1)
 				)

Commit message: CHA: rev 1.2 - der C3 liegt falsch
Connections:
- net at Q9.2 (E), R4.1: now also C4.1
- net at C3.1, Q13.3 (C), Q9.1 (B)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: no longer C4.1
Changed lines of the file:
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@@
 		(title "Audio Amp")
 		(date "2025-04-29")
-		(rev "1.1")
+		(rev "1.2")
 		(company "Lucca Kuvecke, Marcel Tanneberger")
 	)
@@
 	)
 	(junction
+		(at 186.69 118.11)
+		(diameter 0)
+		(color 0 0 0 0)
+	)
+	(junction
 		(at 177.8 81.28)
 		(diameter 0)
@@
 	(wire
 		(pts
-			(xy 175.26 111.76) (xy 175.26 120.65)
-		)
-		(stroke
-			(width 0)
-			(type default)
-		)
-	)
-	(wire
-		(pts
 			(xy 58.42 99.06) (xy 58.42 105.41)
 		)
@@
 	(wire
 		(pts
+			(xy 175.26 120.65) (xy 175.26 118.11)
+		)
+		(stroke
+			(width 0)
+			(type default)
+		)
+	)
+	(wire
+		(pts
 			(xy 74.93 90.17) (xy 74.93 105.41)
 		)
@@
 	(wire
 		(pts
+			(xy 186.69 118.11) (xy 186.69 120.65)
+		)
+		(stroke
+			(width 0)
+			(type default)
+		)
+	)
+	(wire
+		(pts
 			(xy 93.98 100.33) (xy 93.98 105.41)
 		)
@@
 	(wire
 		(pts
-			(xy 186.69 116.84) (xy 186.69 120.65)
-		)
-		(stroke
+			(xy 175.26 118.11) (xy 186.69 118.11)
+		)
+		(stroke
+			(width 0)
+			(type default)
+		)
+	)
+	(wire
+		(pts
+			(xy 186.69 116.84) (xy 186.69 118.11)
+		)
+		(stroke
